Commit message: add imu serial node

File: urdf/robot.urdf (robot description, URDF)
Before this commit: robot robot, 3 links, 2 joints
Links:
- link base_link: geometry collision box size=0.35 0.24 0.15; collision sphere radius=0.0175
Joints:
- joint joint_left_wheel: origin xyz=0 0.165 0 rpy=0 0 0 -> xyz=0 0.135 0.035 rpy=0 0 0
- joint joint_right_wheel: origin xyz=0 -0.165 0 rpy=0 0 0 -> xyz=0 -0.135 0.035 rpy=0 0 0
